File: Motor Board/Motor Board.kicad_pcb (KiCad board)
At the start: 2 copper layers, 39.5 x 34.5 mm, 28 parts, among them J1 Programmer, J2 Gecko, M1 26M048B2U Stepper, U1 ULN2003A, U2 PIC18F26K83, U3 MCP2562, U4 INA180

Commit message: Finish schematics and footprint assignments
Parts:
- removed C1, C2, C3: 0.1uF, Capacitor_SMD:C_0805_2012Metric_Pad1.18x1.45mm_HandSolder
- removed D1: RED, LED_SMD:LED_1206_3216Metric_Pad1.42x1.75mm_HandSolder
- removed D2: BLUE, LED_SMD:LED_1206_3216Metric_Pad1.42x1.75mm_HandSolder
- removed D3: WHITE, LED_SMD:LED_1206_3216Metric_Pad1.42x1.75mm_HandSolder
- removed F1: Polyfuse 350mA, Fuse:Fuse_1206_3216Metric_Pad1.42x1.75mm_HandSolder
- removed G***: LOGO, Downloaded:Waterloo Rocketry Logo
- removed H1, H2, H3, H4: Mount, MountingHole:MountingHole_3.2mm_M3_Pad
- removed J1: Programmer, Downloaded:GCT_BG300-05-X-X-A_REVC
- removed J2: Gecko, Downloaded:G125-MH10605M4R
- removed M1: 26M048B2U Stepper, Downloaded:G125-MH10605M4R
- removed PWM1, PWM2, PWM3, PWM4: TestPoint, TestPoint:TestPoint_THTPad_1.0x1.0mm_Drill0.5mm
- removed R1: 10k, Resistor_SMD:R_0805_2012Metric_Pad1.20x1.40mm_HandSolder
- removed R2: 220R, Resistor_SMD:R_0805_2012Metric_Pad1.20x1.40mm_HandSolder
- removed R3, R4: 120R, Resistor_SMD:R_0805_2012Metric_Pad1.20x1.40mm_HandSolder
- removed R5: 62mR, Resistor_SMD:R_0805_2012Metric_Pad1.20x1.40mm_HandSolder
- removed U1: ULN2003A, Downloaded:DIP-16_STM
- removed U2: PIC18F26K83, Downloaded:SOIC28_SO_MCH
- removed U3: MCP2562, Package_SO:SOIC-8_3.9x4.9mm_P1.27mm
- removed U4: INA180, Package_TO_SOT_SMD:SOT-23-5_HandSoldering
Routing:
- net /PWM4: track 81.0 -> 0.00 mm, vias 2 -> 0
- net GND: track 74.6 -> 0.00 mm, vias 4 -> 0
- net +5V: track 70.0 -> 0.00 mm, vias 3 -> 0
- net +12V: track 63.0 -> 0.00 mm
- net /PWM3: track 62.0 -> 0.00 mm, vias 2 -> 0
- net /PWM2: track 56.1 -> 0.00 mm
- net Net-(U2-RA2): track 45.7 -> 0.00 mm, vias 3 -> 0
- net Net-(U4-IN+): track 41.7 -> 0.00 mm, vias 2 -> 0
- net Net-(U2-RA0): track 33.2 -> 0.00 mm, vias 3 -> 0
- net /PWM1: track 32.6 -> 0.00 mm
- net /~{MCLR}: track 31.5 -> 0.00 mm, vias 2 -> 0
- net /CANH: track 31.3 -> 0.00 mm
- net Net-(D1-K): track 25.5 -> 0.00 mm, vias 1 -> 0
- net Net-(U2-RA1): track 25.1 -> 0.00 mm, vias 1 -> 0
- net /CURR_SENS: track 22.3 -> 0.00 mm, vias 2 -> 0
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- removed copper zone on F.Cu, net +5V
- removed copper zone on B.Cu, net GND
Other:
- board outline removed
- board text removed: "Step on me Connor S"

Commit message: Add osc to motor
Parts:
- added C1: 0.1uF, Capacitor_SMD:C_0805_2012Metric_Pad1.18x1.45mm_HandSolder, F.Cu at (134.0, 94.0)
- added C2: 0.1uF, Capacitor_SMD:C_0805_2012Metric_Pad1.18x1.45mm_HandSolder, F.Cu at (138.8, 94.0)
- added C3: 0.1uF, Capacitor_SMD:C_0805_2012Metric_Pad1.18x1.45mm_HandSolder, F.Cu at (143.5, 94.0)
- added C4: 27pF, Capacitor_SMD:C_0805_2012Metric_Pad1.18x1.45mm_HandSolder, B.Cu at (145.5, 77.2)
- added C5: 27pF, Capacitor_SMD:C_0805_2012Metric_Pad1.18x1.45mm_HandSolder, B.Cu at (145.5, 81.0)
- added D1: RED, LED_SMD:LED_1206_3216Metric_Pad1.42x1.75mm_HandSolder, F.Cu at (137.9, 63.9)
- added D2: BLUE, LED_SMD:LED_1206_3216Metric_Pad1.42x1.75mm_HandSolder, F.Cu at (128.1, 68.6)
- added D3: WHITE, LED_SMD:LED_1206_3216Metric_Pad1.42x1.75mm_HandSolder, F.Cu at (148.6, 68.6)
- added F1: Polyfuse 350mA, Fuse:Fuse_1206_3216Metric_Pad1.42x1.75mm_HandSolder, B.Cu at (144.9, 71.9)
- added H1: Mount, MountingHole:MountingHole_3.2mm_M3_Pad, F.Cu at (124.0, 61.5)
- added H2: Mount, MountingHole:MountingHole_3.2mm_M3_Pad, F.Cu at (152.5, 61.5)
- added H3: Mount, MountingHole:MountingHole_3.2mm_M3_Pad, F.Cu at (124.0, 91.5)
- added H4: Mount, MountingHole:MountingHole_3.2mm_M3_Pad, F.Cu at (152.5, 91.5)
- added J1: Programmer, Canhw:PinSocket_5x2.54_SMD_90deg_952-3198-1-ND, B.Cu at (133.4, 84.8)
- added J2: Gecko, Canhw:connector_Harwin_G125–MG10605M4P, F.Cu at (149.5, 78.0)
- added J3: Gecko, Canhw:connector_Harwin_G125–MG10605M4P, F.Cu at (127.0, 78.0)
- added J4: Conn_01x02_Socket, Connector_JST:JST_PH_S2B-PH-K_1x02_P2.00mm_Horizontal, F.Cu at (132.5, 65.0)
- added J5: Conn_01x02_Socket, Connector_JST:JST_PH_S2B-PH-K_1x02_P2.00mm_Horizontal, F.Cu at (146.0, 65.0)
- added Q1: BSS316NN, Package_TO_SOT_SMD:SOT-323_SC-70, B.Cu at (138.8, 77.0)
- added R1: 10k, Resistor_SMD:R_0805_2012Metric_Pad1.20x1.40mm_HandSolder, F.Cu at (144.0, 90.0)
- added R2: 220R, Resistor_SMD:R_0805_2012Metric_Pad1.20x1.40mm_HandSolder, F.Cu at (135.0, 90.0)
- added R3: 120R, Resistor_SMD:R_0805_2012Metric_Pad1.20x1.40mm_HandSolder, F.Cu at (138.0, 90.0)
- added R4: 120R, Resistor_SMD:R_0805_2012Metric_Pad1.20x1.40mm_HandSolder, F.Cu at (141.0, 90.0)
- added R5: 62mR, Resistor_SMD:R_0805_2012Metric_Pad1.20x1.40mm_HandSolder, F.Cu at (132.0, 90.0)
- added R6: 10kR, Resistor_SMD:R_0805_2012Metric_Pad1.20x1.40mm_HandSolder, F.Cu at (147.0, 90.0)
- added R7: 10kR, Resistor_SMD:R_0805_2012Metric_Pad1.20x1.40mm_HandSolder, F.Cu at (129.0, 90.0)
- added U2: PIC18F26K83, Package_SO:SOIC-28W_7.5x18.7mm_P1.27mm, F.Cu at (138.0, 78.2)
- added U3: MCP2562, Package_SO:SOIC-8_3.9x4.9mm_P1.27mm, B.Cu at (138.5, 72.4)
- added U4: INA180, Package_TO_SOT_SMD:SOT-23-5_HandSoldering, B.Cu at (138.8, 81.2)
- added Y1: 12MHz Crystal, Crystal:Crystal_HC49-4H_Vertical, B.Cu at (137.9, 61.1)
Routing:
- net GND: track 0.00 -> 81.2 mm, vias 0 -> 6
- net Net-(D1-K): track 0.00 -> 50.2 mm, vias 0 -> 4
- net /LIM_1: track 0.00 -> 42.4 mm, vias 0 -> 2
- net /LIM_2: track 0.00 -> 40.6 mm
- net Net-(D2-K): track 0.00 -> 38.8 mm, vias 0 -> 2
- net Net-(D3-K): track 0.00 -> 33.1 mm, vias 0 -> 2
- net +5V: track 0.00 -> 31.2 mm
- net Net-(U4-IN+): track 0.00 -> 28.0 mm, vias 0 -> 3
- net /OSC2: track 0.00 -> 28.0 mm, vias 0 -> 1
- net /OSC1: track 0.00 -> 26.5 mm, vias 0 -> 1
- net Net-(J2-Pin_5): track 0.00 -> 20.9 mm
- net /CANL: track 0.00 -> 19.4 mm, vias 0 -> 1
- net /CANH: track 0.00 -> 17.8 mm, vias 0 -> 1
- net Net-(U2-RA2): track 0.00 -> 10.3 mm
- net /MTR_ON: track 0.00 -> 9.39 mm, vias 0 -> 1
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- added copper zone on F.Cu, net +5V
- added copper zone on B.Cu, net GND
Other:
- board outline added: 37.5 x 39 mm
- board text added: "CANBUS"
- board text added: "SERVO"
