File: Sensor Board/Sensor Board.kicad_pcb (KiCad board)
At the start: 4 copper layers, 41.7 x 49.5 mm, 61 parts, among them J1 Programming Header, J2 CAN Bus Connector, J3 Micro_SD_Card, U1 PIC18F26K83, U2 INA180, U3 MCP2562, U4 OPA323, U5 MCP3561-E/ST, U6 SPX3819M5-L-3-3, U7 MCP1501-30xSN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

Commit message: Polish PCB; gerbs
Parts:
- C3: moved to F.Cu
- moved C3 9.27 mm to (203.1, 98.0), turned to 180 degrees
- moved C21 9.25 mm to (209.0, 86.9)
- moved C11 8.10 mm to (213.0, 89.6), turned to 180 degrees
- moved C9 6.92 mm to (209.1, 84.6), turned to 180 degrees
- moved U6 6.02 mm to (213.1, 86.1)
- moved U2 4.21 mm to (209.1, 81.0)
- moved C8 4.20 mm to (206.2, 81.0)
- moved R12 4.20 mm to (212.5, 80.9)
- moved F1 3.56 mm to (220.0, 85.7)
- moved J2 3.54 mm to (216.8, 87.2), turned to 90 degrees
- moved R4 2.05 mm to (200.9, 100.1)
- moved C20 1.02 mm to (215.9, 67.1)
- moved D1 0.78 mm to (217.8, 58.7)
- moved C22 0.64 mm to (215.9, 69.2)
- moved R1 0.41 mm to (205.4, 64.0)
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Routing:
- net +5V: track 68.2 -> 79.0 mm
- net +3V3D: track 31.1 -> 41.0 mm, vias 20 -> 10
- net Net-(U2-IN+): track 7.94 -> 16.2 mm
- net /CANH: track 20.5 -> 12.2 mm
- net /CANL: track 23.0 -> 15.1 mm
- net AGND: track 7.32 -> 9.74 mm, vias 48 -> 47
- net /MOSI: track 35.1 -> 37.3 mm
- net (no net): track 2.03 -> 0.00 mm
- net /CURR_SENSE: track 6.62 -> 5.24 mm
- net Net-(U6-BP): track 3.30 -> 2.21 mm
- net /CANRX: track 25.6 -> 26.7 mm
- net GND: track 21.0 -> 20.1 mm, vias 44 -> 41
- net Net-(J2-Pin_5): track 2.67 -> 1.93 mm
- net Net-(D1-A): track 10.7 -> 9.95 mm
- net /CANTX: track 28.8 -> 29.4 mm
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Other:
- board text removed: "HOT!"

Commit message: removed random 3v3 plane left behine and reconnected grunds
Routing:
- net (no net): track 0.00 -> 1.40 mm
- net +3V3D: vias 10 -> 9
- removed copper zone on B.Cu, net +3V3D
Changed lines of the file:
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@@
 			(size 3.8 3.8)
 			(drill 2.25)
-			(layers "*.Cu" "*.Mask")
+			(layers "*.Cu" "*.Mask" "In3.Cu" "In4.Cu" "In5.Cu" "In6.Cu" "In7.Cu" "In8.Cu"
+				"In9.Cu" "In10.Cu" "In11.Cu" "In12.Cu" "In13.Cu" "In14.Cu" "In15.Cu"
+				"In16.Cu" "In17.Cu" "In18.Cu" "In19.Cu" "In20.Cu" "In21.Cu" "In22.Cu"
+				"In23.Cu" "In24.Cu" "In25.Cu" "In26.Cu" "In27.Cu" "In28.Cu" "In29.Cu"
+				"In30.Cu"
+			)
 			(remove_unused_layers no)
 		)
@@
 			(size 3.8 3.8)
 			(drill 2.25)
-			(layers "*.Cu" "*.Mask")
+			(layers "*.Cu" "*.Mask" "In3.Cu" "In4.Cu" "In5.Cu" "In6.Cu" "In7.Cu" "In8.Cu"
+				"In9.Cu" "In10.Cu" "In11.Cu" "In12.Cu" "In13.Cu" "In14.Cu" "In15.Cu"
+				"In16.Cu" "In17.Cu" "In18.Cu" "In19.Cu" "In20.Cu" "In21.Cu" "In22.Cu"
+				"In23.Cu" "In24.Cu" "In25.Cu" "In26.Cu" "In27.Cu" "In28.Cu" "In29.Cu"
+				"In30.Cu"
+			)
 			(remove_unused_layers no)
 		)
@@
 			(size 1 1)
 			(drill 0.6)
-			(layers "*.Cu" "*.Mask")
+			(layers "*.Cu" "*.Mask" "In3.Cu" "In4.Cu" "In5.Cu" "In6.Cu" "In7.Cu" "In8.Cu"
+				"In9.Cu" "In10.Cu" "In11.Cu" "In12.Cu" "In13.Cu" "In14.Cu" "In15.Cu"
+				"In16.Cu" "In17.Cu" "In18.Cu" "In19.Cu" "In20.Cu" "In21.Cu" "In22.Cu"
+				"In23.Cu" "In24.Cu" "In25.Cu" "In26.Cu" "In27.Cu" "In28.Cu" "In29.Cu"
+				"In30.Cu"
+			)
 			(remove_unused_layers no)
 			(net 44 "unconnected-(J2-Pin_1-Pad1)")
@@
 			(size 1 1)
 			(drill 0.6)
-			(layers "*.Cu" "*.Mask")
+			(layers "*.Cu" "*.Mask" "In3.Cu" "In4.Cu" "In5.Cu" "In6.Cu" "In7.Cu" "In8.Cu"
+				"In9.Cu" "In10.Cu" "In11.Cu" "In12.Cu" "In13.Cu" "In14.Cu" "In15.Cu"
+				"In16.Cu" "In17.Cu" "In18.Cu" "In19.Cu" "In20.Cu" "In21.Cu" "In22.Cu"
+				"In23.Cu" "In24.Cu" "In25.Cu" "In26.Cu" "In27.Cu" "In28.Cu" "In29.Cu"
+				"In30.Cu"
+			)
 			(remove_unused_layers no)
 			(net 29 "/CANL")
@@
 			(size 1 1)
 			(drill 0.6)
-			(layers "*.Cu" "*.Mask")
+			(layers "*.Cu" "*.Mask" "In3.Cu" "In4.Cu" "In5.Cu" "In6.Cu" "In7.Cu" "In8.Cu"
+				"In9.Cu" "In10.Cu" "In11.Cu" "In12.Cu" "In13.Cu" "In14.Cu" "In15.Cu"
+				"In16.Cu" "In17.Cu" "In18.Cu" "In19.Cu" "In20.Cu" "In21.Cu" "In22.Cu"
+				"In23.Cu" "In24.Cu" "In25.Cu" "In26.Cu" "In27.Cu" "In28.Cu" "In29.Cu"
+				"In30.Cu"
+			)
 			(remove_unused_layers no)
 			(net 30 "/CANH")
@@
 			(size 1 1)
 			(drill 0.6)
-			(layers "*.Cu" "*.Mask")
+			(layers "*.Cu" "*.Mask" "In3.Cu" "In4.Cu" "In5.Cu" "In6.Cu" "In7.Cu" "In8.Cu"
+				"In9.Cu" "In10.Cu" "In11.Cu" "In12.Cu" "In13.Cu" "In14.Cu" "In15.Cu"
+				"In16.Cu" "In17.Cu" "In18.Cu" "In19.Cu" "In20.Cu" "In21.Cu" "In22.Cu"
+				"In23.Cu" "In24.Cu" "In25.Cu" "In26.Cu" "In27.Cu" "In28.Cu" "In29.Cu"
+				"In30.Cu"
+			)
 			(remove_unused_layers no)
 			(net 54 "GND")
@@
 			(size 1 1)
 			(drill 0.6)
-			(layers "*.Cu" "*.Mask")
+			(layers "*.Cu" "*.Mask" "In3.Cu" "In4.Cu" "In5.Cu" "In6.Cu" "In7.Cu" "In8.Cu"
+				"In9.Cu" "In10.Cu" "In11.Cu" "In12.Cu" "In13.Cu" "In14.Cu" "In15.Cu"
+				"In16.Cu" "In17.Cu" "In18.Cu" "In19.Cu" "In20.Cu" "In21.Cu" "In22.Cu"
+				"In23.Cu" "In24.Cu" "In25.Cu" "In26.Cu" "In27.Cu" "In28.Cu" "In29.Cu"
+				"In30.Cu"
+			)
 			(remove_unused_layers no)
 			(net 34 "Net-(J2-Pin_5)")
@@
 			(size 1 1)
 			(drill 0.6)
-			(layers "*.Cu" "*.Mask")
+			(layers "*.Cu" "*.Mask" "In3.Cu" "In4.Cu" "In5.Cu" "In6.Cu" "In7.Cu" "In8.Cu"
+				"In9.Cu" "In10.Cu" "In11.Cu" "In12.Cu" "In13.Cu" "In14.Cu" "In15.Cu"
+				"In16.Cu" "In17.Cu" "In18.Cu" "In19.Cu" "In20.Cu" "In21.Cu" "In22.Cu"
+				"In23.Cu" "In24.Cu" "In25.Cu" "In26.Cu" "In27.Cu" "In28.Cu" "In29.Cu"
+				"In30.Cu"
+			)
 			(remove_unused_layers no)
 			(net 45 "unconnected-(J2-Pin_6-Pad6)")
@@
 		(tags "capacitor handsolder")
 		(property "Reference" "C16"
-			(at -0.1281 -1.32 270)
+			(at -0.1281 -1.32 -90)
 			(layer "F.SilkS")
 			(effects
@@
 		(tags "capacitor handsolder")
 		(property "Reference" "C15"
-			(at 0.0293 1.3716 270)
+			(at 0.0293 1.3716 -90)
 			(layer "F.SilkS")
 			(effects
@@
 			(size 5.6 5.6)
 			(drill 3.2)
-			(layers "*.Cu" "*.Mask")
+			(layers "*.Cu" "*.Mask" "In3.Cu" "In4.Cu" "In5.Cu" "In6.Cu" "In7.Cu" "In8.Cu"
+				"In9.Cu" "In10.Cu" "In11.Cu" "In12.Cu" "In13.Cu" "In14.Cu" "In15.Cu"
+				"In16.Cu" "In17.Cu" "In18.Cu" "In19.Cu" "In20.Cu" "In21.Cu" "In22.Cu"
+				"In23.Cu" "In24.Cu" "In25.Cu" "In26.Cu" "In27.Cu" "In28.Cu" "In29.Cu"
+				"In30.Cu"
+			)
 			(remove_unused_layers no)
 			(net 16 "AGND")
@@
 			(size 5.6 5.6)
 			(drill 3.2)
-			(layers "*.Cu" "*.Mask")
+			(layers "*.Cu" "*.Mask" "In3.Cu" "In4.Cu" "In5.Cu" "In6.Cu" "In7.Cu" "In8.Cu"
+				"In9.Cu" "In10.Cu" "In11.Cu" "In12.Cu" "In13.Cu" "In14.Cu" "In15.Cu"
+				"In16.Cu" "In17.Cu" "In18.Cu" "In19.Cu" "In20.Cu" "In21.Cu" "In22.Cu"
+				"In23.Cu" "In24.Cu" "In25.Cu" "In26.Cu" "In27.Cu" "In28.Cu" "In29.Cu"
+				"In30.Cu"
+			)
 			(remove_unused_layers no)
 			(net 54 "GND")
@@
 			(size 5.6 5.6)
 			(drill 3.2)
-			(layers "*.Cu" "*.Mask")
+			(layers "*.Cu" "*.Mask" "In3.Cu" "In4.Cu" "In5.Cu" "In6.Cu" "In7.Cu" "In8.Cu"
+				"In9.Cu" "In10.Cu" "In11.Cu" "In12.Cu" "In13.Cu" "In14.Cu" "In15.Cu"
+				"In16.Cu" "In17.Cu" "In18.Cu" "In19.Cu" "In20.Cu" "In21.Cu" "In22.Cu"
+				"In23.Cu" "In24.Cu" "In25.Cu" "In26.Cu" "In27.Cu" "In28.Cu" "In29.Cu"
+				"In30.Cu"
+			)
 			(remove_unused_layers no)
 			(net 54 "GND")
@@
 			)
 			(height -4.3)
-			(gr_text "141.7323 mils"
+			(gr_text "3.6000 mm"
 				(at 210.7796 63.7748 0)
 				(layer "Dwgs.User")
@@
 			)
 			(height 1.4)
-			(gr_text "141.7323 mils"
+			(gr_text "3.6000 mm"
 				(at 206.4296 58.8248 90)
 				(layer "Dwgs.User")
@@
 			(size 5.6 5.6)
 			(drill 3.2)
-			(layers "*.Cu" "*.Mask")
+			(layers "*.Cu" "*.Mask" "In3.Cu" "In4.Cu" "In5.Cu" "In6.Cu" "In7.Cu" "In8.Cu"
+				"In9.Cu" "In10.Cu" "In11.Cu" "In12.Cu" "In13.Cu" "In14.Cu" "In15.Cu"
+				"In16.Cu" "In17.Cu" "In18.Cu" "In19.Cu" "In20.Cu" "In21.Cu" "In22.Cu"
+				"In23.Cu" "In24.Cu" "In25.Cu" "In26.Cu" "In27.Cu" "In28.Cu" "In29.Cu"
+				"In30.Cu"
+			)
 			(remove_unused_layers no)
 			(net 54 "GND")
@@
 			(size 1.5 1.5)
 			(drill 0.8)
-			(layers "*.Cu" "*.Mask")
+			(layers "*.Cu" "*.Mask" "In3.Cu" "In4.Cu" "In5.Cu" "In6.Cu" "In7.Cu" "In8.Cu"
+				"In9.Cu" "In10.Cu" "In11.Cu" "In12.Cu" "In13.Cu" "In14.Cu" "In15.Cu"
+				"In16.Cu" "In17.Cu" "In18.Cu" "In19.Cu" "In20.Cu" "In21.Cu" "In22.Cu"
+				"In23.Cu" "In24.Cu" "In25.Cu" "In26.Cu" "In27.Cu" "In28.Cu" "In29.Cu"
+				"In30.Cu"
+			)
 			(remove_unused_layers no)
 			(net 1 "/OSC1")
@@
 			(size 1.5 1.5)
 			(drill 0.8)
-			(layers "*.Cu" "*.Mask")
+			(layers "*.Cu" "*.Mask" "In3.Cu" "In4.Cu" "In5.Cu" "In6.Cu" "In7.Cu" "In8.Cu"
+				"In9.Cu" "In10.Cu" "In11.Cu" "In12.Cu" "In13.Cu" "In14.Cu" "In15.Cu"
+				"In16.Cu" "In17.Cu" "In18.Cu" "In19.Cu" "In20.Cu" "In21.Cu" "In22.Cu"
+				"In23.Cu" "In24.Cu" "In25.Cu" "In26.Cu" "In27.Cu" "In28.Cu" "In29.Cu"
+				"In30.Cu"
+			)
 			(remove_unused_layers no)
 			(net 2 "/OSC2")
@@
 		(tags "test point SMD pad rectangle square")
 		(property "Reference" "3V3A"
-			(at -1.778 -0.1016 270)
+			(at -1.778 -0.1016 -90)
 			(layer "F.SilkS")
 			(effects
@@
 		(tags "capacitor handsolder")
 		(property "Reference" "C11"
-			(at -0.0801 -1.778 360)
+			(at -0.0801 -1.778 0)
 			(layer "B.SilkS")
 			(effects
@@
 		)
 		(property "Value" "10nF"
-			(at 0 -1.68 360)
+			(at 0 -1.68 0)
 			(layer "B.Fab")
 			(effects
@@
 		)
 		(fp_text user "${REFERENCE}"
-			(at 0 0 360)
+			(at 0 0 0)
 			(layer "B.Fab")
 			(effects
@@
 		(tags "capacitor handsolder")
 		(property "Reference" "C9"
-			(at 2.8233 0 360)
+			(at 2.8233 0 0)
 			(layer "B.SilkS")
 			(effects
@@
 		)
 		(property "Value" "1uF"
-			(at 0 -1.68 360)
+			(at 0 -1.68 0)
 			(layer "B.Fab")
 			(effects
@@
 		)
 		(fp_text user "${REFERENCE}"
-			(at 0 0 360)
+			(at 0 0 0)
 			(layer "B.Fab")
 			(effects
@@
 		(height -5.1)
 		(orientation 1)
-		(gr_text "1475.1969 mils"
+		(gr_text "37.4700 mm"
 			(at 123.5 83.235 90)
 			(layer "Dwgs.User")
@@
 		(height 8.63)
 		(orientation 0)
-		(gr_text "1669.7835 mils"
+		(gr_text "42.4125 mm"
 			(at 151.60625 108.8 0)
 			(layer "Dwgs.User")
@@
 	)
 	(segment
+		(start 189.992 57.785)
+		(end 191.389 57.785)
+		(width 0.762)
+		(layer "In1.Cu")
+		(net 0)
+	)
+	(segment
 		(start 189.72 86.8315)
 		(end 189.72 88.247)
@@
 	)
 	(via
-		(at 212.598 99.314)
-		(size 0.6)
-		(drill 0.3)
-		(layers "F.Cu" "B.Cu")
-		(free yes)
-		(net 3)
-	)
-	(via
 		(at 189.738 60.706)
 		(size 0.762)
@@
 			)
 		)
-	)
-	(zone
-		(net 3)
-		(net_name "+3V3D")
-		(layer "B.Cu")
-		(hatch edge 0.5)
-		(priority 6)
-		(connect_pads
-			(clearance 0.5)
-		)
-		(min_thickness 0.25)
-		(filled_areas_thickness no)
-		(fill yes
-			(thermal_gap 0.5)
-			(thermal_bridge_width 0.5)
-		)
-		(polygon
-			(pts
-				(xy 212.09 91.44) (xy 212.09 99.568) (xy 217.424 99.568) (xy 217.424 91.44)
-			)
-		)
